Commit message: grip 확인 후 재시도 기능 추가

File: install/ur_moveit_config/share/ur_moveit_config/srdf/ur_macro.srdf.xacro (robot description, xacro)
@@ -64,4 +64,5 @@
     <disable_collisions link1="gripper_robotiq_85_right_finger_link"     link2="gripper_robotiq_85_right_knuckle_link"       reason="Never"/>
     <disable_collisions link1="gripper_robotiq_85_right_finger_tip_link" link2="gripper_robotiq_85_right_inner_knuckle_link" reason="Never"/>
-  </xacro:macro>
+    <disable_collisions link1="tool0" link2="gripper_robotiq_85_left_knuckle_joint" reason="adjacent"/>
+    </xacro:macro>
 </robot>

File: install/ur_simulation_gz/share/ur_simulation_gz/urdf/ur_gz.urdf.xacro (robot description, xacro)
@@ -68,5 +68,5 @@
       sim_ignition="true"
       >
-      <origin xyz="0 0 0.01" rpy="0 0 0"/>
+      <origin xyz="0 0 0.005" rpy="0 0 0"/>
   </xacro:robotiq_gripper>
   <gazebo reference="world">
