Commit message: moveit cpp 제어 test 성공 ur_sim_control_launch.py, ur_sim_moveit_launch.py 에서 name 파라미터 부분 수정했음

File: install/ur_moveit_config/share/ur_moveit_config/srdf/ur.srdf.xacro (robot description, xacro)
@@ -1,11 +1 @@
-<?xml version="1.0" encoding="UTF-8"?>
-<robot xmlns:xacro="http://wiki.ros.org/xacro" name="$(arg name)">
-  <!-- robot name parameter -->
-  <xacro:arg name="name" default="ur"/>
-  <xacro:include filename="$(find ur_moveit_config)/srdf/ur_macro.srdf.xacro"/>
-  <xacro:ur_srdf/>
-  <group name="gripper">
-    <joint name="gripper_robotiq_85_left_knuckle_joint"/>
-  </group>
-  <end_effector name="gripper" parent_link="tool0" group="gripper"/>
-</robot>
+/home/bin1225/workspaces/ur_gz/src/ur_moveit_config/srdf/ur.srdf.xacro

File: install/ur_moveit_config/share/ur_moveit_config/srdf/ur_macro.srdf.xacro (robot description, xacro)
@@ -1,56 +1 @@
-<?xml version="1.0" encoding="UTF-8"?>
-<robot xmlns:xacro="http://wiki.ros.org/xacro">
-<!--This does not replace URDF, and is not an extension of URDF.
-    This is a format for representing semantic information about the robot structure.
-    A URDF file must exist for this robot as well, where the joints and the links that are referenced are defined
--->
-  <xacro:macro name="ur_srdf" params="">
-    <!--GROUPS - Representation of a set of joints and links. This can be useful for specifying DOF to plan for, defining arms, end effectors, etc-->
-    <!--LINKS - When a link is specified, the parent joint of that link (if it exists) is automatically included-->
-    <!--JOINTS - When a joint is specified, the child link of that joint (which will always exist) is automatically included-->
-    <!--CHAINS - When a chain is specified, all the links along the chain (including endpoints) are included in the group. Additionally, all the joints that are parents to included links are also included. This means that joints along the chain and the parent joint of the base link are included in the group-->
-    <!--SUBGROUPS - Groups can also be formed by referencing to already defined group names-->
-    <group name="ur_manipulator">
-      <chain base_link="base_link" tip_link="tool0" />
-    </group>
-    <!--GROUP STATES - Purpose - Define a named state for a particular group, in terms of joint values. This is useful to define states like 'folded arms'-->
-    <group_state name="home" group="ur_manipulator">
-      <joint name="elbow_joint" value="0" />
-      <joint name="shoulder_lift_joint" value="-1.5707" />
-      <joint name="shoulder_pan_joint" value="0" />
-      <joint name="wrist_1_joint" value="0" />
-      <joint name="wrist_2_joint" value="0" />
-      <joint name="wrist_3_joint" value="0" />
-    </group_state>
-    <group_state name="up" group="ur_manipulator">
-      <joint name="elbow_joint" value="0" />
-      <joint name="shoulder_lift_joint" value="-1.5707" />
-      <joint name="shoulder_pan_joint" value="0" />
-      <joint name="wrist_1_joint" value="-1.5707" />
-      <joint name="wrist_2_joint" value="0" />
-      <joint name="wrist_3_joint" value="0" />
-    </group_state>
-    <group_state name="test_configuration" group="ur_manipulator">
-      <joint name="elbow_joint" value="1.4" />
-      <joint name="shoulder_lift_joint" value="-1.62" />
-      <joint name="shoulder_pan_joint" value="1.54" />
-      <joint name="wrist_1_joint" value="-1.2" />
-      <joint name="wrist_2_joint" value="-1.6" />
-      <joint name="wrist_3_joint" value="-0.11" />
-    </group_state>
-    <!--END EFFECTOR - Purpose - Represent information about an end effector.-->
-    <!--VIRTUAL JOINT - Purpose - this element defines a virtual joint between a robot link and an external frame of reference (considered fixed with respect to the robot)-->
-    <!--DISABLE COLLISIONS - By default it is assumed that any link of the robot could potentially come into collision with any other link in the robot. This tag disables collision checking between a specified pair of links. -->
-    <disable_collisions link1="base_link" link2="base_link_inertia" reason="Adjacent" />
-    <disable_collisions link1="base_link_inertia" link2="shoulder_link" reason="Adjacent" />
-    <disable_collisions link1="tool0" link2="wrist_1_link" reason="Never" />
-    <disable_collisions link1="tool0" link2="wrist_2_link" reason="Never" />
-    <disable_collisions link1="tool0" link2="wrist_3_link" reason="Adjacent" />
-    <disable_collisions link1="forearm_link" link2="upper_arm_link" reason="Adjacent" />
-    <disable_collisions link1="forearm_link" link2="wrist_1_link" reason="Adjacent" />
-    <disable_collisions link1="shoulder_link" link2="upper_arm_link" reason="Adjacent" />
-    <disable_collisions link1="wrist_1_link" link2="wrist_2_link" reason="Adjacent" />
-    <disable_collisions link1="wrist_1_link" link2="wrist_3_link" reason="Never" />
-    <disable_collisions link1="wrist_2_link" link2="wrist_3_link" reason="Adjacent" />
-  </xacro:macro>
-</robot>
+/home/bin1225/workspaces/ur_gz/src/ur_moveit_config/srdf/ur_macro.srdf.xacro

File: install/ur_simulation_gz/share/ur_simulation_gz/urdf/ur_gz.ros2_control.xacro (robot description, xacro)
@@ -1,23 +1 @@
-<?xml version="1.0"?>
-<robot xmlns:xacro="http://www.ros.org/wiki/xacro">
-  <xacro:include filename="$(find ur_description)/urdf/inc/ur_joint_control.xacro" />
-  <xacro:macro name="ur_ros2_control" params="
-    name
-    tf_prefix
-    transmission_hw_interface:=hardware_interface/PositionJointInterface
-    initial_positions:=${dict(shoulder_pan_joint=0.0,shoulder_lift_joint=-1.57,elbow_joint=0.0,wrist_1_joint=-1.57,wrist_2_joint=0.0,wrist_3_joint=0.0)}
-    ">
-    <!-- Add URDF transmission elements (for ros_control) -->
-    <!--<xacro:ur_arm_transmission prefix="${prefix}" hw_interface="${transmission_hw_interface}" />-->
-    <!-- Placeholder for ros2_control transmission which don't yet exist -->
-    <ros2_control name="${name}" type="system">
-      <hardware>
-        <plugin>gz_ros2_control/GazeboSimSystem</plugin>
-      </hardware>
-      <xacro:ur_joint_control_description
-        tf_prefix="${tf_prefix}"
-        initial_positions="${initial_positions}"
-      />
-    </ros2_control>
-  </xacro:macro>
-</robot>
+/home/bin1225/workspaces/ur_gz/src/ur_simulation_gz/ur_simulation_gz/urdf/ur_gz.ros2_control.xacro

File: install/ur_simulation_gz/share/ur_simulation_gz/urdf/ur_gz.urdf.xacro (robot description, xacro)
@@ -1,88 +1 @@
-<?xml version="1.0"?>
-<robot xmlns:xacro="http://wiki.ros.org/xacro" name="$(arg name)">
-  <!-- robot name parameter -->
-  <xacro:arg name="name" default="ur"/>
-  <!-- import main macro -->
-  <xacro:include filename="$(find ur_description)/urdf/ur_macro.xacro"/>
-  <xacro:include filename="$(find ur_simulation_gz)/urdf/ur_gz.ros2_control.xacro" />
-  <xacro:include filename="$(find robotiq_description)/urdf/robotiq_2f_85_macro.urdf.xacro"/>
-  <!-- possible 'ur_type' values: ur3, ur3e, ur5, ur5e, ur7e, ur10, ur10e, ur12e, ur16e, ur20, ur30 -->
-  <!-- the default value should raise an error in case this was called without defining the type -->
-  <xacro:arg name="ur_type" default="ur5x"/>
-  <!-- parameters -->
-  <xacro:arg name="tf_prefix" default="" />
-  <xacro:arg name="joint_limit_params" default="$(find ur_description)/config/$(arg ur_type)/joint_limits.yaml"/>
-  <xacro:arg name="kinematics_params" default="$(find ur_description)/config/$(arg ur_type)/default_kinematics.yaml"/>
-  <xacro:arg name="physical_params" default="$(find ur_description)/config/$(arg ur_type)/physical_parameters.yaml"/>
-  <xacro:arg name="visual_params" default="$(find ur_description)/config/$(arg ur_type)/visual_parameters.yaml"/>
-  <xacro:arg name="transmission_hw_interface" default=""/>
-  <xacro:arg name="safety_limits" default="false"/>
-  <xacro:arg name="safety_pos_margin" default="0.15"/>
-  <xacro:arg name="safety_k_position" default="20"/>
-  <xacro:arg name="simulation_controllers" default="" />
-  <xacro:arg name="ros_namespace" default="" />
-  <!-- create link fixed to the "world" -->
-  <link name="world" />
-  <link name="ground_plane">
-    <visual>
-      <origin rpy="0 0 0" xyz="0 0 0"/>
-      <geometry>
-        <box size="5 5 0"/>
-      </geometry>
-      <material name="ground_white">
-        <color rgba="1 1 1 0.5"/>
-      </material>
-    </visual>
-    <collision>
-      <origin rpy="0 0 0" xyz="0 0 0"/>
-      <geometry>
-        <box size="5 5 0"/>
-      </geometry>
-    </collision>
-  </link>
-  <joint name="ground_plane_joint" type="fixed">
-    <origin xyz="0 0 -0.01" rpy="0 0 0"/>
-    <parent link="world"/>
-    <child link="ground_plane"/>
-  </joint>
-  <!-- arm -->
-  <xacro:ur_robot
-    name="$(arg name)"
-    tf_prefix="$(arg tf_prefix)"
-    parent="world"
-    joint_limits_parameters_file="$(arg joint_limit_params)"
-    kinematics_parameters_file="$(arg kinematics_params)"
-    physical_parameters_file="$(arg physical_params)"
-    visual_parameters_file="$(arg visual_params)"
-    safety_limits="$(arg safety_limits)"
-    safety_pos_margin="$(arg safety_pos_margin)"
-    safety_k_position="$(arg safety_k_position)"
-    force_abs_paths="true"
-    >
-    <origin xyz="0 0 0" rpy="0 0 0" />          <!-- position robot in the world -->
-  </xacro:ur_robot>
-   <xacro:robotiq_gripper
-      name="RobotiqGripperHardwareInterface"
-      parent="$(arg tf_prefix)tool0"
-      prefix="gripper_"
-      sim_ignition="true"
-      >
-      <origin xyz="0 0 0" rpy="0 0 0"/>
-  </xacro:robotiq_gripper>
-  <gazebo reference="world">
-  </gazebo>
-  <gazebo>
-    <plugin filename="gz_ros2_control-system" name="gz_ros2_control::GazeboSimROS2ControlPlugin">
-      <parameters>$(arg simulation_controllers)</parameters>
-      <ros>
-        <namespace>$(arg ros_namespace)</namespace>
-      </ros>
-    </plugin>
-  </gazebo>
-  <!-- ros2 control instance -->
-  <xacro:ur_ros2_control
-    name="$(arg name)"
-    tf_prefix="$(arg tf_prefix)"
-    transmission_hw_interface="$(arg transmission_hw_interface)"
-  />
-</robot>
+/home/bin1225/workspaces/ur_gz/src/ur_simulation_gz/ur_simulation_gz/urdf/ur_gz.urdf.xacro

Commit message: moveit arg로 좌표 넘겨 위치 이동 시키기

File: install/ur_moveit_config/share/ur_moveit_config/srdf/ur.srdf.xacro (robot description, xacro)
@@ -1 +1,11 @@
-/home/bin1225/workspaces/ur_gz/src/ur_moveit_config/srdf/ur.srdf.xacro
+<?xml version="1.0" encoding="UTF-8"?>
+<robot xmlns:xacro="http://wiki.ros.org/xacro" name="$(arg name)">
+  <!-- robot name parameter -->
+  <xacro:arg name="name" default="ur"/>
+  <xacro:include filename="$(find ur_moveit_config)/srdf/ur_macro.srdf.xacro"/>
+  <xacro:ur_srdf/>
+  <group name="gripper">
+    <joint name="gripper_robotiq_85_left_knuckle_joint"/>
+  </group>
+  <end_effector name="gripper" parent_link="tool0" group="gripper"/>
+</robot>

File: install/ur_moveit_config/share/ur_moveit_config/srdf/ur_macro.srdf.xacro (robot description, xacro)
@@ -1 +1,67 @@
-/home/bin1225/workspaces/ur_gz/src/ur_moveit_config/srdf/ur_macro.srdf.xacro
+<?xml version="1.0" encoding="UTF-8"?>
+<robot xmlns:xacro="http://wiki.ros.org/xacro">
+<!--This does not replace URDF, and is not an extension of URDF.
+    This is a format for representing semantic information about the robot structure.
+    A URDF file must exist for this robot as well, where the joints and the links that are referenced are defined
+-->
+  <xacro:macro name="ur_srdf" params="">
+    <!--GROUPS - Representation of a set of joints and links. This can be useful for specifying DOF to plan for, defining arms, end effectors, etc-->
+    <!--LINKS - When a link is specified, the parent joint of that link (if it exists) is automatically included-->
+    <!--JOINTS - When a joint is specified, the child link of that joint (which will always exist) is automatically included-->
+    <!--CHAINS - When a chain is specified, all the links along the chain (including endpoints) are included in the group. Additionally, all the joints that are parents to included links are also included. This means that joints along the chain and the parent joint of the base link are included in the group-->
+    <!--SUBGROUPS - Groups can also be formed by referencing to already defined group names-->
+    <group name="ur_manipulator">
+      <chain base_link="base_link" tip_link="tool0" />
+    </group>
+    <!--GROUP STATES - Purpose - Define a named state for a particular group, in terms of joint values. This is useful to define states like 'folded arms'-->
+    <group_state name="home" group="ur_manipulator">
+      <joint name="elbow_joint" value="0" />
+      <joint name="shoulder_lift_joint" value="-1.5707" />
+      <joint name="shoulder_pan_joint" value="0" />
+      <joint name="wrist_1_joint" value="0" />
+      <joint name="wrist_2_joint" value="0" />
+      <joint name="wrist_3_joint" value="0" />
+    </group_state>
+    <group_state name="up" group="ur_manipulator">
+      <joint name="elbow_joint" value="0" />
+      <joint name="shoulder_lift_joint" value="-1.5707" />
+      <joint name="shoulder_pan_joint" value="0" />
+      <joint name="wrist_1_joint" value="-1.5707" />
+      <joint name="wrist_2_joint" value="0" />
+      <joint name="wrist_3_joint" value="0" />
+    </group_state>
+    <group_state name="test_configuration" group="ur_manipulator">
+      <joint name="elbow_joint" value="1.4" />
+      <joint name="shoulder_lift_joint" value="-1.62" />
+      <joint name="shoulder_pan_joint" value="1.54" />
+      <joint name="wrist_1_joint" value="-1.2" />
+      <joint name="wrist_2_joint" value="-1.6" />
+      <joint name="wrist_3_joint" value="-0.11" />
+    </group_state>
+    <!--END EFFECTOR - Purpose - Represent information about an end effector.-->
+    <!--VIRTUAL JOINT - Purpose - this element defines a virtual joint between a robot link and an external frame of reference (considered fixed with respect to the robot)-->
+    <!--DISABLE COLLISIONS - By default it is assumed that any link of the robot could potentially come into collision with any other link in the robot. This tag disables collision checking between a specified pair of links. -->
+    <disable_collisions link1="base_link" link2="base_link_inertia" reason="Adjacent" />
+    <disable_collisions link1="base_link_inertia" link2="shoulder_link" reason="Adjacent" />
+    <disable_collisions link1="tool0" link2="wrist_1_link" reason="Never" />
+    <disable_collisions link1="tool0" link2="wrist_2_link" reason="Never" />
+    <disable_collisions link1="tool0" link2="wrist_3_link" reason="Adjacent" />
+    <disable_collisions link1="forearm_link" link2="upper_arm_link" reason="Adjacent" />
+    <disable_collisions link1="forearm_link" link2="wrist_1_link" reason="Adjacent" />
+    <disable_collisions link1="shoulder_link" link2="upper_arm_link" reason="Adjacent" />
+    <disable_collisions link1="wrist_1_link" link2="wrist_2_link" reason="Adjacent" />
+    <disable_collisions link1="wrist_1_link" link2="wrist_3_link" reason="Never" />
+    <disable_collisions link1="wrist_2_link" link2="wrist_3_link" reason="Adjacent" />
+    <!-- 추가: gripper self-collision 무시 -->
+    <disable_collisions link1="gripper_robotiq_85_base_link"      link2="gripper_robotiq_85_left_inner_knuckle_link"   reason="Never"/>
+    <disable_collisions link1="gripper_robotiq_85_base_link"      link2="gripper_robotiq_85_left_knuckle_link"         reason="Never"/>
+    <disable_collisions link1="gripper_robotiq_85_base_link"      link2="gripper_robotiq_85_right_inner_knuckle_link"  reason="Never"/>
+    <disable_collisions link1="gripper_robotiq_85_base_link"      link2="gripper_robotiq_85_right_knuckle_link"        reason="Never"/>
+    <disable_collisions link1="gripper_robotiq_85_left_finger_link"      link2="gripper_robotiq_85_left_finger_tip_link"     reason="Never"/>
+    <disable_collisions link1="gripper_robotiq_85_left_finger_link"      link2="gripper_robotiq_85_left_knuckle_link"        reason="Never"/>
+    <disable_collisions link1="gripper_robotiq_85_left_finger_tip_link"  link2="gripper_robotiq_85_left_inner_knuckle_link" reason="Never"/>
+    <disable_collisions link1="gripper_robotiq_85_right_finger_link"     link2="gripper_robotiq_85_right_finger_tip_link"    reason="Never"/>
+    <disable_collisions link1="gripper_robotiq_85_right_finger_link"     link2="gripper_robotiq_85_right_knuckle_link"       reason="Never"/>
+    <disable_collisions link1="gripper_robotiq_85_right_finger_tip_link" link2="gripper_robotiq_85_right_inner_knuckle_link" reason="Never"/>
+  </xacro:macro>
+</robot>

File: install/ur_simulation_gz/share/ur_simulation_gz/urdf/ur_gz.urdf.xacro (robot description, xacro)
@@ -1 +1,88 @@
-/home/bin1225/workspaces/ur_gz/src/ur_simulation_gz/ur_simulation_gz/urdf/ur_gz.urdf.xacro
+<?xml version="1.0"?>
+<robot xmlns:xacro="http://wiki.ros.org/xacro" name="$(arg name)">
+  <!-- robot name parameter -->
+  <xacro:arg name="name" default="ur"/>
+  <!-- import main macro -->
+  <xacro:include filename="$(find ur_description)/urdf/ur_macro.xacro"/>
+  <xacro:include filename="$(find ur_simulation_gz)/urdf/ur_gz.ros2_control.xacro" />
+  <xacro:include filename="$(find robotiq_description)/urdf/robotiq_2f_85_macro.urdf.xacro"/>
+  <!-- possible 'ur_type' values: ur3, ur3e, ur5, ur5e, ur7e, ur10, ur10e, ur12e, ur16e, ur20, ur30 -->
+  <!-- the default value should raise an error in case this was called without defining the type -->
+  <xacro:arg name="ur_type" default="ur5x"/>
+  <!-- parameters -->
+  <xacro:arg name="tf_prefix" default="" />
+  <xacro:arg name="joint_limit_params" default="$(find ur_description)/config/$(arg ur_type)/joint_limits.yaml"/>
+  <xacro:arg name="kinematics_params" default="$(find ur_description)/config/$(arg ur_type)/default_kinematics.yaml"/>
+  <xacro:arg name="physical_params" default="$(find ur_description)/config/$(arg ur_type)/physical_parameters.yaml"/>
+  <xacro:arg name="visual_params" default="$(find ur_description)/config/$(arg ur_type)/visual_parameters.yaml"/>
+  <xacro:arg name="transmission_hw_interface" default=""/>
+  <xacro:arg name="safety_limits" default="false"/>
+  <xacro:arg name="safety_pos_margin" default="0.15"/>
+  <xacro:arg name="safety_k_position" default="20"/>
+  <xacro:arg name="simulation_controllers" default="" />
+  <xacro:arg name="ros_namespace" default="" />
+  <!-- create link fixed to the "world" -->
+  <link name="world" />
+  <link name="ground_plane">
+    <visual>
+      <origin rpy="0 0 0" xyz="0 0 0"/>
+      <geometry>
+        <box size="5 5 0"/>
+      </geometry>
+      <material name="ground_white">
+        <color rgba="1 1 1 0.5"/>
+      </material>
+    </visual>
+    <collision>
+      <origin rpy="0 0 0" xyz="0 0 0"/>
+      <geometry>
+        <box size="5 5 0"/>
+      </geometry>
+    </collision>
+  </link>
+  <joint name="ground_plane_joint" type="fixed">
+    <origin xyz="0 0 -0.01" rpy="0 0 0"/>
+    <parent link="world"/>
+    <child link="ground_plane"/>
+  </joint>
+  <!-- arm -->
+  <xacro:ur_robot
+    name="$(arg name)"
+    tf_prefix="$(arg tf_prefix)"
+    parent="world"
+    joint_limits_parameters_file="$(arg joint_limit_params)"
+    kinematics_parameters_file="$(arg kinematics_params)"
+    physical_parameters_file="$(arg physical_params)"
+    visual_parameters_file="$(arg visual_params)"
+    safety_limits="$(arg safety_limits)"
+    safety_pos_margin="$(arg safety_pos_margin)"
+    safety_k_position="$(arg safety_k_position)"
+    force_abs_paths="true"
+    >
+    <origin xyz="0 0 0" rpy="0 0 0" />          <!-- position robot in the world -->
+  </xacro:ur_robot>
+   <xacro:robotiq_gripper
+      name="RobotiqGripperHardwareInterface"
+      parent="$(arg tf_prefix)tool0"
+      prefix="gripper_"
+      sim_ignition="true"
+      >
+      <origin xyz="0 0 0.01" rpy="0 0 0"/>
+  </xacro:robotiq_gripper>
+  <gazebo reference="world">
+  </gazebo>
+  <gazebo>
+    <plugin filename="gz_ros2_control-system" name="gz_ros2_control::GazeboSimROS2ControlPlugin">
+      <parameters>$(arg simulation_controllers)</parameters>
+      <ros>
+        <namespace>$(arg ros_namespace)</namespace>
+      </ros>
+    </plugin>
+  </gazebo>
+  <!-- ros2 control instance -->
+  <xacro:ur_ros2_control
+    name="$(arg name)"
+    tf_prefix="$(arg tf_prefix)"
+    transmission_hw_interface="$(arg transmission_hw_interface)"
+  />
+</robot>

File: install/ur_simulation_gz/share/ur_simulation_gz/urdf/ur_gz_setup_test.urdf.xacro (robot description, xacro)
@@ -1 +1,59 @@
-/home/bin1225/workspaces/ur_gz/src/ur_simulation_gz/ur_simulation_gz/urdf/ur_gz_setup_test.urdf.xacro
+<?xml version="1.0"?>
+<robot name="ur5e_simple" xmlns="http://www.ros.org/wiki/robot_model" xmlns:xacro="http://www.ros.org/wiki/xacro">
+  <!-- 1 base_link -->
+  <link name="base_link"/>
+  <!-- 2 shoulder_pan_joint -->
+  <link name="shoulder_link"/>
+  <joint name="shoulder_pan_joint" type="continuous">
+    <parent link="base_link"/>
+    <child  link="shoulder_link"/>
+    <axis  xyz="0 0 1"/>
+  </joint>
+  <!-- 3 shoulder_lift_joint -->
+  <link name="upper_arm_link"/>
+  <joint name="shoulder_lift_joint" type="continuous">
+    <parent link="shoulder_link"/>
+    <child  link="upper_arm_link"/>
+    <axis  xyz="0 1 0"/>
+  </joint>
+  <!-- 4 elbow_joint -->
+  <link name="forearm_link"/>
+  <joint name="elbow_joint" type="continuous">
+    <parent link="upper_arm_link"/>
+    <child  link="forearm_link"/>
+    <axis  xyz="0 1 0"/>
+  </joint>
+  <!-- 5 wrist_1_joint -->
+  <link name="wrist_1_link"/>
+  <joint name="wrist_1_joint" type="continuous">
+    <parent link="forearm_link"/>
+    <child  link="wrist_1_link"/>
+    <axis  xyz="0 1 0"/>
+  </joint>
+  <!-- 6 wrist_2_joint -->
+  <link name="wrist_2_link"/>
+  <joint name="wrist_2_joint" type="continuous">
+    <parent link="wrist_1_link"/>
+    <child  link="wrist_2_link"/>
+    <axis  xyz="0 0 1"/>
+  </joint>
+  <!-- 7 wrist_3_joint -->
+  <link name="wrist_3_link"/>
+  <joint name="wrist_3_joint" type="continuous">
+    <parent link="wrist_2_link"/>
+    <child  link="wrist_3_link"/>
+    <axis  xyz="0 1 0"/>
+  </joint>
+  <!-- 8 tool0 (end effector mounting) -->
+  <link name="tool0"/>
+  <joint name="tool0_joint" type="fixed">
+    <parent link="wrist_3_link"/>
+    <child  link="tool0"/>
+  </joint>
+  <!-- 9 gripper (rigidly attached) -->
+  <link name="gripper"/>
+  <joint name="gripper_fixed_joint" type="fixed">
+    <parent link="tool0"/>
+    <child  link="gripper"/>
+  </joint>
+</robot>
