Commit message: namespace 조정 전 저장

File: src/ur_moveit_config/srdf/dual.srdf.xacro (robot description, xacro)
@@ -1,16 +1,7 @@
-<?xml version="1.0" encoding="UTF-8"?>
+<?xml version="1.0"?>
 <robot xmlns:xacro="http://wiki.ros.org/xacro" name="$(arg name)">
-  <!-- robot name parameter -->
-  <xacro:arg name="name" default="ur"/>
-  <xacro:arg name="prefix" default=""/>
-  <xacro:property name="prefix" value="$(arg prefix)"/>
-  <xacro:include filename="$(find ur_moveit_config)/srdf/dual_macro.srdf.xacro"/>
-  <xacro:ur_srdf prefix="$(arg prefix)"/>
-  <group name="gripper">
-    <!-- ★ joint 이름에도 prefix -->
-    <joint name="${prefix}gripper_robotiq_85_left_knuckle_joint"/>
-  </group>
-  <end_effector name="gripper"
-                parent_link="${prefix}tool0"
-                group="gripper"/>
+  <xacro:arg name="name" default=""/>
+  <xacro:include filename="/home/bin1225/workspaces/ur_gz/src/ur_moveit_config/srdf/dual_macro.srdf.xacro"/>
+  <xacro:arg name="tf_prefix" default="" />
+  <xacro:ur_srdf tf_prefix="$(arg tf_prefix)" />
 </robot>

File: src/ur_moveit_config/srdf/dual_macro.srdf.xacro (robot description, xacro)
@@ -1,81 +1,89 @@
 <?xml version="1.0" encoding="UTF-8"?>
 <robot xmlns:xacro="http://wiki.ros.org/xacro">
-  <!-- ★ macro 파라미터에 prefix 추가 -->
-  <xacro:macro name="ur_srdf" params="prefix">
+  <!-- ★ macro 파라미터에 tf_prefix 추가 -->
+  <xacro:macro name="ur_srdf" params="tf_prefix">
     <!--──────────── GROUPS ────────────-->
-    <group name="ur_manipulator">
-      <chain base_link="${prefix}base_link" tip_link="${prefix}tool0"/>
-    </group>
+  <group name="${tf_prefix}manipulator">
+    <chain base_link="${tf_prefix}base_link" tip_link="${tf_prefix}tool0"/>
+  </group>
+  <group name="${tf_prefix}gripper">
+    <joint name="${tf_prefix}gripper_robotiq_85_left_knuckle_joint"/>
+  </group>
+  <end_effector
+    name="${tf_prefix}gripper"
+    parent_link="${tf_prefix}tool0"
+    group="${tf_prefix}gripper"/>
+  <!-- ... 기존 내용 ... -->
     <!--──────────── GROUP STATES ──────-->
-    <group_state name="home" group="ur_manipulator">
-      <joint name="${prefix}elbow_joint"          value="0"/>
-      <joint name="${prefix}shoulder_lift_joint"  value="-1.5707"/>
-      <joint name="${prefix}shoulder_pan_joint"   value="0"/>
-      <joint name="${prefix}wrist_1_joint"        value="0"/>
-      <joint name="${prefix}wrist_2_joint"        value="0"/>
-      <joint name="${prefix}wrist_3_joint"        value="0"/>
+    <group_state name="home" group="${tf_prefix}manipulator">
+      <joint name="${tf_prefix}elbow_joint"          value="0"/>
+      <joint name="${tf_prefix}shoulder_lift_joint"  value="-1.5707"/>
+      <joint name="${tf_prefix}shoulder_pan_joint"   value="0"/>
+      <joint name="${tf_prefix}wrist_1_joint"        value="0"/>
+      <joint name="${tf_prefix}wrist_2_joint"        value="0"/>
+      <joint name="${tf_prefix}wrist_3_joint"        value="0"/>
     </group_state>
-    <group_state name="up" group="ur_manipulator">
-      <joint name="${prefix}elbow_joint"         value="0"/>
-      <joint name="${prefix}shoulder_lift_joint" value="-1.5707"/>
-      <joint name="${prefix}shoulder_pan_joint"  value="0"/>
-      <joint name="${prefix}wrist_1_joint"       value="-1.5707"/>
-      <joint name="${prefix}wrist_2_joint"       value="0"/>
-      <joint name="${prefix}wrist_3_joint"       value="0"/>
+    <group_state name="up" group="${tf_prefix}manipulator">
+      <joint name="${tf_prefix}elbow_joint"         value="0"/>
+      <joint name="${tf_prefix}shoulder_lift_joint" value="-1.5707"/>
+      <joint name="${tf_prefix}shoulder_pan_joint"  value="0"/>
+      <joint name="${tf_prefix}wrist_1_joint"       value="-1.5707"/>
+      <joint name="${tf_prefix}wrist_2_joint"       value="0"/>
+      <joint name="${tf_prefix}wrist_3_joint"       value="0"/>
     </group_state>
-    <group_state name="test_configuration" group="ur_manipulator">
-      <joint name="${prefix}elbow_joint"         value="1.4"/>
-      <joint name="${prefix}shoulder_lift_joint" value="-1.62"/>
-      <joint name="${prefix}shoulder_pan_joint"  value="1.54"/>
-      <joint name="${prefix}wrist_1_joint"       value="-1.2"/>
-      <joint name="${prefix}wrist_2_joint"       value="-1.6"/>
-      <joint name="${prefix}wrist_3_joint"       value="-0.11"/>
+    <group_state name="test_configuration" group="${tf_prefix}manipulator">
+      <joint name="${tf_prefix}elbow_joint"         value="1.4"/>
+      <joint name="${tf_prefix}shoulder_lift_joint" value="-1.62"/>
+      <joint name="${tf_prefix}shoulder_pan_joint"  value="1.54"/>
+      <joint name="${tf_prefix}wrist_1_joint"       value="-1.2"/>
+      <joint name="${tf_prefix}wrist_2_joint"       value="-1.6"/>
+      <joint name="${tf_prefix}wrist_3_joint"       value="-0.11"/>
     </group_state>
     <!--──────────── DISABLE COLLISIONS ─-->
-    <disable_collisions link1="${prefix}base_link"
-                        link2="${prefix}base_link_inertia" reason="Adjacent"/>
-    <disable_collisions link1="${prefix}base_link_inertia"
-                        link2="${prefix}shoulder_link"      reason="Adjacent"/>
-    <disable_collisions link1="${prefix}tool0"
-                        link2="${prefix}wrist_1_link"       reason="Never"/>
-    <disable_collisions link1="${prefix}tool0"
-                        link2="${prefix}wrist_2_link"       reason="Never"/>
-    <disable_collisions link1="${prefix}tool0"
-                        link2="${prefix}wrist_3_link"       reason="Adjacent"/>
-    <disable_collisions link1="${prefix}forearm_link"
-                        link2="${prefix}upper_arm_link"     reason="Adjacent"/>
-    <disable_collisions link1="${prefix}forearm_link"
-                        link2="${prefix}wrist_1_link"       reason="Adjacent"/>
-    <disable_collisions link1="${prefix}shoulder_link"
-                        link2="${prefix}upper_arm_link"     reason="Adjacent"/>
-    <disable_collisions link1="${prefix}wrist_1_link"
-                        link2="${prefix}wrist_2_link"       reason="Adjacent"/>
-    <disable_collisions link1="${prefix}wrist_1_link"
-                        link2="${prefix}wrist_3_link"       reason="Never"/>
-    <disable_collisions link1="${prefix}wrist_2_link"
-                        link2="${prefix}wrist_3_link"       reason="Adjacent"/>
-    <!-- gripper self-collision 무시 (모두 prefix) -->
-    <disable_collisions link1="${prefix}gripper_robotiq_85_base_link"
-                        link2="${prefix}gripper_robotiq_85_left_inner_knuckle_link" reason="Never"/>
-    <disable_collisions link1="${prefix}gripper_robotiq_85_base_link"
-                        link2="${prefix}gripper_robotiq_85_left_knuckle_link"       reason="Never"/>
-    <disable_collisions link1="${prefix}gripper_robotiq_85_base_link"
-                        link2="${prefix}gripper_robotiq_85_right_inner_knuckle_link" reason="Never"/>
-    <disable_collisions link1="${prefix}gripper_robotiq_85_base_link"
-                        link2="${prefix}gripper_robotiq_85_right_knuckle_link"      reason="Never"/>
-    <disable_collisions link1="${prefix}gripper_robotiq_85_left_finger_link"
-                        link2="${prefix}gripper_robotiq_85_left_finger_tip_link"     reason="Never"/>
-    <disable_collisions link1="${prefix}gripper_robotiq_85_left_finger_link"
-                        link2="${prefix}gripper_robotiq_85_left_knuckle_link"        reason="Never"/>
-    <disable_collisions link1="${prefix}gripper_robotiq_85_left_finger_tip_link"
-                        link2="${prefix}gripper_robotiq_85_left_inner_knuckle_link"  reason="Never"/>
-    <disable_collisions link1="${prefix}gripper_robotiq_85_right_finger_link"
-                        link2="${prefix}gripper_robotiq_85_right_finger_tip_link"    reason="Never"/>
-    <disable_collisions link1="${prefix}gripper_robotiq_85_right_finger_link"
-                        link2="${prefix}gripper_robotiq_85_right_knuckle_link"       reason="Never"/>
-    <disable_collisions link1="${prefix}gripper_robotiq_85_right_finger_tip_link"
-                        link2="${prefix}gripper_robotiq_85_right_inner_knuckle_link" reason="Never"/>
-    <disable_collisions link1="${prefix}tool0"
-                        link2="${prefix}gripper_robotiq_85_left_knuckle_joint"
+    <disable_collisions link1="${tf_prefix}base_link"
+                        link2="${tf_prefix}base_link_inertia" reason="Adjacent"/>
+    <disable_collisions link1="${tf_prefix}base_link_inertia"
+                        link2="${tf_prefix}shoulder_link"      reason="Adjacent"/>
+    <disable_collisions link1="${tf_prefix}tool0"
+                        link2="${tf_prefix}wrist_1_link"       reason="Never"/>
+    <disable_collisions link1="${tf_prefix}tool0"
+                        link2="${tf_prefix}wrist_2_link"       reason="Never"/>
+    <disable_collisions link1="${tf_prefix}tool0"
+                        link2="${tf_prefix}wrist_3_link"       reason="Adjacent"/>
+    <disable_collisions link1="${tf_prefix}forearm_link"
+                        link2="${tf_prefix}upper_arm_link"     reason="Adjacent"/>
+    <disable_collisions link1="${tf_prefix}forearm_link"
+                        link2="${tf_prefix}wrist_1_link"       reason="Adjacent"/>
+    <disable_collisions link1="${tf_prefix}shoulder_link"
+                        link2="${tf_prefix}upper_arm_link"     reason="Adjacent"/>
+    <disable_collisions link1="${tf_prefix}wrist_1_link"
+                        link2="${tf_prefix}wrist_2_link"       reason="Adjacent"/>
+    <disable_collisions link1="${tf_prefix}wrist_1_link"
+                        link2="${tf_prefix}wrist_3_link"       reason="Never"/>
+    <disable_collisions link1="${tf_prefix}wrist_2_link"
+                        link2="${tf_prefix}wrist_3_link"       reason="Adjacent"/>
+    <!-- gripper self-collision 무시 (모두 tf_prefix) -->
+    <disable_collisions link1="${tf_prefix}gripper_robotiq_85_base_link"
+                        link2="${tf_prefix}gripper_robotiq_85_left_inner_knuckle_link" reason="Never"/>
+    <disable_collisions link1="${tf_prefix}gripper_robotiq_85_base_link"
+                        link2="${tf_prefix}gripper_robotiq_85_left_knuckle_link"       reason="Never"/>
+    <disable_collisions link1="${tf_prefix}gripper_robotiq_85_base_link"
+                        link2="${tf_prefix}gripper_robotiq_85_right_inner_knuckle_link" reason="Never"/>
+    <disable_collisions link1="${tf_prefix}gripper_robotiq_85_base_link"
+                        link2="${tf_prefix}gripper_robotiq_85_right_knuckle_link"      reason="Never"/>
+    <disable_collisions link1="${tf_prefix}gripper_robotiq_85_left_finger_link"
+                        link2="${tf_prefix}gripper_robotiq_85_left_finger_tip_link"     reason="Never"/>
+    <disable_collisions link1="${tf_prefix}gripper_robotiq_85_left_finger_link"
+                        link2="${tf_prefix}gripper_robotiq_85_left_knuckle_link"        reason="Never"/>
+    <disable_collisions link1="${tf_prefix}gripper_robotiq_85_left_finger_tip_link"
+                        link2="${tf_prefix}gripper_robotiq_85_left_inner_knuckle_link"  reason="Never"/>
+    <disable_collisions link1="${tf_prefix}gripper_robotiq_85_right_finger_link"
+                        link2="${tf_prefix}gripper_robotiq_85_right_finger_tip_link"    reason="Never"/>
+    <disable_collisions link1="${tf_prefix}gripper_robotiq_85_right_finger_link"
+                        link2="${tf_prefix}gripper_robotiq_85_right_knuckle_link"       reason="Never"/>
+    <disable_collisions link1="${tf_prefix}gripper_robotiq_85_right_finger_tip_link"
+                        link2="${tf_prefix}gripper_robotiq_85_right_inner_knuckle_link" reason="Never"/>
+    <disable_collisions link1="${tf_prefix}tool0"
+                        link2="${tf_prefix}gripper_robotiq_85_left_knuckle_link"
                         reason="adjacent"/>
   </xacro:macro>
